File: light-driver/light-driver.kicad_pcb (KiCad board)
At the start: 2 copper layers, 59 parts, among them J1 LED-strip0, J2 Power/CAN, J3 LED-strip1, J4 Power/CAN, J5 SWD, J6 Conn_01x08_Pin, J7 ARGB, Q1 IRLML0030, Q2 IRLML0030, Q3 IRLML0030, Q4 IRLML0030, U1 TC1185-xCT, U2 TPP361061-T6TR, U3 TJA1051T-3, U4 STM32G0B1KETx

Commit message: Finish light-driver hardware
Parts:
- added C15: 100n, Capacitor_SMD:C_0603_1608Metric_Pad1.08x0.95mm_HandSolder, F.Cu at (85.7, 97.3)
- added C16: 100n, Capacitor_SMD:C_0603_1608Metric_Pad1.08x0.95mm_HandSolder, F.Cu at (81.9, 104.1)
- added J8: Conn_01x04_Pin, Connector_PinSocket_2.00mm:PinSocket_1x04_P2.00mm_Vertical, F.Cu at (110.0, 98.5)
- C1, C10, C11, C12, C13, C14, C2, C3, C5, C7, C8, C9, D1, D4, D5, D6, J5, L1, R1, R2, R4, R5, R6, R7, U2: moved to B.Cu
- C4, C6: footprint Capacitor_SMD:C_0805_2012Metric_Pad1.18x1.45mm_HandSolder -> Capacitor_SMD:C_0603_1608Metric_Pad1.08x0.95mm_HandSolder; moved to B.Cu
- U1: footprint Package_TO_SOT_SMD:SOT-23-5 -> Package_TO_SOT_SMD:SOT-23-5_HandSoldering; moved to B.Cu
- moved Q1 94.9 mm to (65.8, 101.4), turned to -90 degrees
- moved R11 94.2 mm to (65.8, 97.7), turned to 180 degrees
- moved R10 92.3 mm to (67.8, 96.0), turned to 180 degrees
- moved Q2 92.0 mm to (69.6, 101.4), turned to -90 degrees
- moved R13 90.1 mm to (69.6, 97.7), turned to 180 degrees
- moved R12 88.2 mm to (71.5, 96.0), turned to 180 degrees
- moved R15 86.7 mm to (75.5, 97.8), turned to 180 degrees
- moved R17 86.6 mm to (79.2, 97.8), turned to 180 degrees
- moved Q3 86.0 mm to (75.5, 101.5), turned to -90 degrees
- moved R14 84.6 mm to (77.3, 96.1), turned to 180 degrees
- moved R16 84.6 mm to (81.2, 96.1), turned to 180 degrees
- moved Q4 84.5 mm to (79.2, 101.5), turned to -90 degrees
- moved J1 82.3 mm to (68.3, 106.0), turned to 180 degrees
- moved U2 82.0 mm to (71.2, 99.4), turned to 180 degrees
- moved L1 77.1 mm to (71.2, 92.6)
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Connections:
- net Net-(J6-Pin_1) renamed /PA0
- net Net-(J6-Pin_2) renamed /PA1
- net Net-(J6-Pin_3) renamed /PA2
- net Net-(J6-Pin_4) renamed /PA3
- net Net-(J6-Pin_5) renamed /PA4
- net Net-(J6-Pin_6) renamed /PA5
- net Net-(J6-Pin_7) renamed /PA6
- net Net-(J6-Pin_8) renamed /PA7
- JP1 pad 2: /adressBit2 -> /adressBit0
- JP3 pad 2: /adressBit0 -> /adressBit2
- U4 pad 18: /LED0_warmWhite -> /Status_LED_Red
- U4 pad 19: /LED0_coldWhite -> /Status_LED_Green
- U4 pad 21: /LED1_warmWhite -> unconnected-(U4-PA10/UCPD1_DBCC2-Pad21)
- U4 pad 22: /LED1_coldWhite -> unconnected-(U4-PA9/PA11-Pad22)
- U4 pad 23: unconnected-(U4-PA10/PA12-Pad23) -> /ledData
- U4 pad 26: /Status_LED_Red -> unconnected-(U4-PA15-Pad26)
- U4 pad 28: /Status_LED_Green -> /LED0_warmWhite
- U4 pad 29: /ledData -> /LED0_coldWhite
- U4 pad 30: unconnected-(U4-PB6-Pad30) -> /LED1_warmWhite
- U4 pad 31: unconnected-(U4-PB7-Pad31) -> /LED1_coldWhite
Routing:
- net GND: track 0.00 -> 83.1 mm, vias 0 -> 76
- net +3V3: track 0.00 -> 68.4 mm, vias 0 -> 6
- net +5V: track 0.00 -> 61.5 mm, vias 0 -> 1
- net /CAN-: track 0.00 -> 41.1 mm, vias 0 -> 2
- net /CAN+: track 0.00 -> 39.1 mm
- net +24V: track 0.00 -> 38.3 mm
- net /LED0_warmWhite: track 0.00 -> 24.5 mm
- net /LED0_coldWhite: track 0.00 -> 20.1 mm
- net /ledClock: track 0.00 -> 18.0 mm
- net /SWCLK: track 0.00 -> 17.2 mm, vias 0 -> 1
- net /CAN_RX: track 0.00 -> 14.8 mm, vias 0 -> 2
- net /PA7: track 0.00 -> 14.4 mm
- net /LED1_warmWhite: track 0.00 -> 13.7 mm
- net /PA6: track 0.00 -> 12.8 mm
- net /PA5: track 0.00 -> 11.2 mm
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- added copper zone on B.Cu, net GND
- added copper zone on F.Cu, net GND
- added copper zone on B.Cu, net Net-(U2-SW)
Other:
- board outline added: 59 x 18 mm
- board text added: "Netz39 e.V"
- board text added: "cyberdesk light-driver v1.0 2025-02 by Max2 (Netz39)"
