File: light-driver/light-driver.kicad_sch (KiCad schematic)
At the start: 47 parts, among them J1 LED-strip0, J2 Power/CAN, J3 LED-strip1, J4 Power/CAN, J5 SWD, J6 Conn_01x08_Pin, J7 ARGB, U1 TC1185-xCT, U2 TPP361061-T6TR, U3 TJA1051T-3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

Commit message: Finish light-driver hardware
Parts:
- added C15, C16: 100n, Capacitor_SMD:C_0603_1608Metric_Pad1.08x0.95mm_HandSolder, symbol Device:C
- added J8: Conn_01x04_Pin, Connector_PinSocket_2.00mm:PinSocket_1x04_P2.00mm_Vertical, symbol Connector:Conn_01x04_Pin
- C4, C6: footprint Capacitor_SMD:C_0805_2012Metric_Pad1.18x1.45mm_HandSolder -> Capacitor_SMD:C_0603_1608Metric_Pad1.08x0.95mm_HandSolder
- U1: footprint Package_TO_SOT_SMD:SOT-23-5 -> Package_TO_SOT_SMD:SOT-23-5_HandSoldering
- renumbered JP3 to JP1, JP1 to JP3
Connections:
- net +3V3: now also C16.1, J8.1 (Pin_1), J8.2 (Pin_2)
- net +5V: now also C15.1
- net GND: now also C15.2, C16.2, J8.3 (Pin_3), J8.4 (Pin_4)
- net LED0_coldWhite: now also U4.29 (PB5); no longer U4.19 (PA9/UCPD1_DBCC1)
- net LED0_warmWhite: now also U4.28 (PB4); no longer U4.18 (PA8)
- net LED1_coldWhite: now also U4.31 (PB7); no longer U4.22 (PA9/PA11)
- net LED1_warmWhite: now also U4.30 (PB6); no longer U4.21 (PA10/UCPD1_DBCC2)
- net Status_LED_Green: now also U4.19 (PA9/UCPD1_DBCC1); no longer U4.28 (PB4)
- net Status_LED_Red: now also U4.18 (PA8); no longer U4.26 (PA15)
- net ledData: now also U4.23 (PA10/PA12); no longer U4.29 (PB5)
- net PA3: now reaches J6.4 (Pin_4), U4.10 (PA3)
- net PA4: now reaches J6.5 (Pin_5), U4.11 (PA4)
- net PA5: now reaches J6.6 (Pin_6), U4.12 (PA5)
- net PA6: now reaches J6.7 (Pin_7), U4.13 (PA6)
- net PA7: now reaches J6.8 (Pin_8), U4.14 (PA7)
- net PA0: now reaches J6.1 (Pin_1), U4.7 (PA0)
- net PA1: now reaches J6.2 (Pin_2), U4.8 (PA1)
- net PA2: now reaches J6.3 (Pin_3), U4.9 (PA2)
Other:
- note added: "<- 5V tolerant"
- note added: "optional connections"
- moved on the sheet: C10, C11, C12, C13, C14, D2, D3, J6, R3, R4, R5, U3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
