File: hardware/control-panel/control-panel.kicad_pcb (KiCad board)
At the start: 2 copper layers, 59 x 18 mm, 51 parts, among them J2 Power/CAN, J4 Power/CAN, J5 SWD, J6 Conn_01x06_Pin, J7 ARGB, SW1 RotaryEncoder_Switch, SW2 RotaryEncoder_Switch, SW3 RotaryEncoder_Switch, SW4 RotaryEncoder_Switch, U1 TC1185-xCT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

Commit message: Update footprints to given in inventory
Parts:
- C11, C13, C2, C3, C4, C6: footprint Capacitor_SMD:C_0603_1608Metric_Pad1.08x0.95mm_HandSolder -> Capacitor_SMD:C_0805_2012Metric_Pad1.18x1.45mm_HandSolder
- L1: footprint Inductor_SMD:L_1008_2520Metric_Pad1.43x2.20mm_HandSolder -> Inductor_SMD:L_1210_3225Metric_Pad1.42x2.65mm_HandSolder
- moved C13 0.60 mm to (84.0, 102.5)
- moved C3 0.45 mm to (71.1, 94.2)
- moved L1 0.29 mm to (65.6, 92.9)
- moved C11 0.20 mm to (86.0, 102.5)
Routing:
- net +3V3: vias 7 -> 6

Commit message: Update some values
Parts:
- R8: value 68R -> 390R
- R9: value 4R7 -> 220R
Changed lines of the file:
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@@
 			(plot_on_all_layers_selection 0x0000000_00000000)
 			(disableapertmacros no)
-			(usegerberextensions no)
+			(usegerberextensions yes)
 			(usegerberattributes yes)
 			(usegerberadvancedattributes yes)
-			(creategerberjobfile yes)
+			(creategerberjobfile no)
 			(dashed_line_dash_ratio 12.000000)
 			(dashed_line_gap_ratio 3.000000)
@@
 			(plotinvisibletext no)
 			(sketchpadsonfab no)
-			(subtractmaskfromsilk no)
+			(subtractmaskfromsilk yes)
 			(outputformat 1)
 			(mirror no)
-			(drillshape 1)
+			(drillshape 0)
 			(scaleselection 1)
-			(outputdirectory "")
+			(outputdirectory "gerber")
 		)
 	)
@@
 			)
 		)
-		(property "Value" "68R"
+		(property "Value" "390R"
 			(at 0 1.43 0)
 			(layer "F.Fab")
@@
 			)
 		)
-		(property "Value" "4R7"
+		(property "Value" "220R"
 			(at 0 1.43 0)
 			(layer "F.Fab")
